File: hw/CANSniftAndShift.sch (EAGLE design)
At the start: 0 parts

Commit message: modified schematics
Parts:
- added C1, C10, C11, C12, C2, C3, C4, C5, C6, C7, C8, C9: 100n, rcl:C-EUC0603
- added C13, C14: 18p, rcl:C-EUC0603
- added IC1: AT32UC3C264C, AT32UC3C264C:AT32UC3C264C
- added Q1: 16MHz, crystal-abracon-abm3-smd:CRYSTAL-ABRACON-ABM7-SMD
Connections:
- new net +3V3: C1.1, C10.1, C2.1, C3.1, C4.1, C5.1, C6.1, C7.1, C8.1, C9.1, IC1G$9.VDDIO1, IC1G$9.VDDIO2, IC1G$9.VDDIO3
- new net +5V: IC1G$9.VDDIN_5
- new net GND: C1.2, C10.2, C11.2, C12.2, C13.2, C14.2, C2.2, C3.2, C4.2, C5.2, C6.2, C7.2, C8.2, C9.2, IC1G$9.GNDANA, IC1G$9.GNDCORE, IC1G$9.GNDIO1, IC1G$9.GNDIO2, IC1G$9.GNDIO3, IC1G$9.GNDPLL
- new net N$1: C12.1, IC1G$9.VDDANA
- new net N$2: C11.1, IC1G$9.VDDCORE
- new net N$3: C13.1, IC1G$5.XIN1/PB30, Q1.P$2
- new net N$4: C14.1, IC1G$5.XOUT1/PB31, Q1.P$1
Other:
- note added: "Quarz: Farnell 2467824"

Commit message: updated lbr and schematics
Parts:
- added C15, C16: 100n, SchlegelAr_Master:C_SMD0402
- added CON4: FCI-10033526-N3212LF, SchlegelAr_Master:FCI-10033526-N3212LF
- added IC7: FT232RL, SchlegelAr_Master:FT232RL
- added R22, R23: 0R, SchlegelAr_Master:R0402
- IC1: value AT32UC3C264C -> (none)
Connections:
- new net +5V_USB: C16.P$1, CON4.VBUS, IC7.!RESET, IC7.VCC, IC7.VCCIO
- new net FTDI_3V3OUT: C15.P$1, IC7.3V3OUT
- new net FTDI_RXD: IC1G$7.MACB_RX_ER/RC0_A0/EBI_NCS1/CANRX0/USART0_TXD/PD27, IC7.RXD
- new net FTDI_TXD: IC1G$7.MACB_RX_DV/TC0_B0/EBI_NCS2/CANTX0/USART0_RXD/PD28, IC7.TXD
- new net N$5: IC7.USBDP, R23.P$2
- new net N$6: IC7.USBDM, R22.P$2
- new net USB_D+: CON4.D+, R23.P$1
- new net USB_D-: CON4.D-, R22.P$1
- net GND: now also C15.P$2, C16.P$2, CON4.GND@1, CON4.GND@2, CON4.GND@3, CON4.GND@4, CON4.GND@5, IC7.GND, IC7.GND@1, IC7.GND@2, IC7.GND@A, IC7.TEST
Other:
- note added: "USB UART Bridge"
