File: hw/CANSniftAndShift.sch (EAGLE design)
At the start: 22 parts, among them CON4 FCI-10033526-N3212LF, IC7 FT232RL, Q1 16MHz

Commit message: modified lbr
Parts:
- added C17, C18: (no value), SchlegelAr_Master:C_SMD0603
- added IC2: (no value), v-reg:78XXL
- added SV1: (no value), con-harting-ml:ML10
- C1, C10, C11, C12, C13, C14, C2, C3, C4, C5, C6, C7, C8, C9: device rcl:C-EUC0603 -> SchlegelAr_Master:C_SMD0603
Connections:
- new net !RESET: IC1G$2.!RESET
- new net +12V: C18.P$2, IC2.IN
- new net CAN0RX: IC1G$6.IISC_IWS/EBI_DATA2/CANRX0/PWM_EXTFAULTS0/PC21
- new net CAN0TX: IC1G$6.USART3_CLK/EBI_DATA3/CANTX0/PWM_EXTFAULTS1/PC22
- new net JTAG_TCK: IC1G$4.CANTX1/TCK/PA0, SV1.1
- new net JTAG_TDI: IC1G$4.PAD_EVT0/CANRX1/TDI/PA1, SV1.9
- new net JTAG_TDO: IC1G$4.PAD_EVT1/SCIF_GCLK0/TDO/PA2, SV1.3
- new net JTAG_TMS: IC1G$4.EXTIN1/SCIF_GCLK1/TMS/PA3, SV1.5
- new net N$13: SV1.6
- new net USB_DM: IC1G$8.USB_DM
- new net USB_DP: IC1G$8.USB_DP
- new net USB_VBUS: IC1G$8.USB_VBUS
- net +3V3: now also C1.P$2, C17.P$2, C2.P$2, C3.P$2, C4.P$2, C5.P$2, IC2.OUT, SV1.4; no longer C1.1, C10.1, C2.1, C3.1, C4.1, C5.1, C6.1, C7.1, C8.1, C9.1
- net GND: now also C1.P$1, C11.P$1, C12.P$1, C13.P$1, C14.P$1, C17.P$1, C18.P$1, C2.P$1, C3.P$1, C4.P$1, C5.P$1, IC2.GND, SV1.10, SV1.2; no longer C1.2, C10.2, C11.2, C12.2, C13.2, C14.2, C2.2, C3.2, C4.2, C5.2, C6.2, C7.2, C8.2, C9.2
- net N$1: now also C12.P$2; no longer C12.1
- net N$2: now also C11.P$2; no longer C11.1
- net N$3: now also C13.P$2; no longer C13.1
- net N$4: now also C14.P$2; no longer C14.1

Commit message: first version of schematic
Parts:
- removed C18: (no value), SchlegelAr_Master:C_SMD0603
- removed IC2: (no value), v-reg:78XXL
- added C19, C20: (no value), SchlegelAr_Master:C_SMD0603
- added CON1: FCI-10033526-N3212LF, SchlegelAr_Master:FCI-10033526-N3212LF
- added IC3, IC4: (no value), SchlegelAr_Master:TJA1050
- added IC5: (no value), v-reg:78XXL
- added JP1, JP2, JP3: JUMPER2, SchlegelAr_Master:JUMPER2
- added R1: (no value), SchlegelAr_Master:R0603
- added R2, R3: 120R, SchlegelAr_Master:R0603
- added S1: (no value), switch-omron:10-XX
- added X1, X2: (no value), con-subd:F09HP
- C17: value (none) -> 10u; device SchlegelAr_Master:C_SMD0603 -> SchlegelAr_Master:C_POL4X4MM
Connections:
- removed net +3V3: C1.P$2, C17.P$2, C2.P$2, C3.P$2, C4.P$2, C5.P$2, IC1G$9.VDDIO1, IC1G$9.VDDIO2, IC1G$9.VDDIO3, IC2.OUT, SV1.4
- removed net +5V_USB: C16.P$1, CON4.VBUS, IC7.!RESET, IC7.VCC, IC7.VCCIO
- removed net N$13: SV1.6
- new net CAN1RX: IC1G$6.CANRX1/USART0_RXD/EBI_SWDE/SP0_NPCS0/PWM_PWMH1/PC15, IC4.RXD
- new net CAN1TX: IC1G$6.CANTX1/USART0_TXD/EBI_CAS/SPI0_NPCS1/PWM_PWML1/PC16, IC4.TXD
- new net CANH0: IC3.CANH, JP2.1, X1.7
- new net CANH1: IC4.CANH, JP3.1, X2.7
- new net CANL0: IC3.CANL, R2.P$1, X1.2
- new net CANL1: IC4.CANL, R3.P$1, X2.2
- new net N$12: C16.P$1, IC7.VCC
- new net N$7: JP2.2, R2.P$2
- new net N$9: JP3.2, R3.P$2
- new net SPI0_MISO: IC1G$7.USART0_RXD/TC0_CLK1/EBI_DATA14/TC1_A0/SPI0_MISO/PD1
- new net SPI0_MOSI: IC1G$7.USART0_TXD/QDEC0_QEPI/EBI_DATA13/TC1_CLK0/SPI0_MOSI/PD0
- new net SPI0_NPCS0: IC1G$7.QDEC0_QEPB/EBI_ADDR0/TC0_B2/SPI0_NPCS0/PD3
- new net SPI0_SCK: IC1G$7.QDC0_QEPA/EBI_DATA15/TC0_CLK2/SPI0_SCK/PD2
- net !RESET: now also R1.P$1, S1.P, S1.P1, SV1.6
- net +12V: now also C20.P$2, IC5.IN; no longer C18.P$2, IC2.IN
- net +5V: now also C1.P$2, C10.P$2, C17.+, C19.P$2, C2.P$2, C3.P$2, C4.P$2, C5.P$2, C6.P$2, C7.P$2, C8.P$2, C9.P$2, CON4.VBUS, IC1G$9.VDDIO1, IC1G$9.VDDIO2, IC1G$9.VDDIO3, IC3.VCC, IC4.VCC, IC5.OUT, IC7.!RESET, IC7.VCCIO, JP1.2, R1.P$2, SV1.4
- net CAN0RX: now also IC3.RXD
- net CAN0TX: now also IC3.TXD
- net GND: now also C10.P$1, C17.-, C19.P$1, C20.P$1, C6.P$1, C7.P$1, C8.P$1, C9.P$1, CON1.GND@1, CON1.GND@2, CON1.GND@3, CON1.GND@4, CON1.GND@5, IC3.GND, IC3.S, IC4.GND, IC4.S, IC5.GND, S1.S, S1.S1; no longer C17.P$1, C18.P$1, IC2.GND
- net USB_DM: now also CON1.D-
- net USB_DP: now also CON1.D+
- net USB_VBUS: now also CON1.VBUS, JP1.1
Other:
- note added: "CAN0 & CAN1"
- note added: "JTAG"
- note added: "SUPPLY"
- note added: "USB Connector"
