File: hw/CANSniftAndShift.sch (EAGLE design)
At the start: 39 parts, among them CON1 FCI-10033526-N3212LF, CON4 FCI-10033526-N3212LF, IC7 FT232RL, Q1 16MHz

Commit message: updated sch
Parts:
- added D1: Z3V6, SchlegelAr_Master:BZG03C15TR3
- C13, C14: value 18p -> 27p
- IC3, IC4: value (none) -> TJA1050
- R1: value (none) -> 10k
Connections:
- new net N$8: D1.A, IC1G$9.VDDIN_33
- net +5V: now also D1.C
Other:
- note added: "CAN0"
- note added: "CAN0RX"
- note added: "CAN0TX"
- note added: "CAN1"
- note added: "CAN1RX"
- note added: "CAN1TX"
- note added: "CANH"
- note added: "CANL"
- note added: "CPU"
- note added: "FTDI"
- note added: "FTDI_RX"
- note added: "FTDI_TX"
- note added: "RX"
- note added: "RXD"
- note added: "TX"
- note added: "TXD"
Changed lines of the file:
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@@
 <part name="C9" library="SchlegelAr_Master" deviceset="C_SMD" device="0603" value="100n"/>
 <part name="C10" library="SchlegelAr_Master" deviceset="C_SMD" device="0603" value="100n"/>
-<part name="C13" library="SchlegelAr_Master" deviceset="C_SMD" device="0603" value="18p"/>
-<part name="C14" library="SchlegelAr_Master" deviceset="C_SMD" device="0603" value="18p"/>
+<part name="C13" library="SchlegelAr_Master" deviceset="C_SMD" device="0603" value="27p"/>
+<part name="C14" library="SchlegelAr_Master" deviceset="C_SMD" device="0603" value="27p"/>
 <part name="C11" library="SchlegelAr_Master" deviceset="C_SMD" device="0603" value="100n"/>
 <part name="C12" library="SchlegelAr_Master" deviceset="C_SMD" device="0603" value="100n"/>
@@
 <part name="JP1" library="SchlegelAr_Master" deviceset="JUMPER2" device=""/>
 <part name="S1" library="switch-omron" deviceset="10-XX" device=""/>
-<part name="R1" library="SchlegelAr_Master" deviceset="R" device="0603"/>
+<part name="R1" library="SchlegelAr_Master" deviceset="R" device="0603" value="10k"/>
 <part name="P+12" library="supply1" deviceset="+5V" device=""/>
 <part name="GND20" library="supply1" deviceset="GND" device=""/>
-<part name="IC3" library="SchlegelAr_Master" deviceset="TJA1050" device=""/>
+<part name="IC3" library="SchlegelAr_Master" deviceset="TJA1050" device="" value="TJA1050"/>
 <part name="U$11" library="SchlegelAr_Master" deviceset="+5V" device=""/>
-<part name="IC4" library="SchlegelAr_Master" deviceset="TJA1050" device=""/>
+<part name="IC4" library="SchlegelAr_Master" deviceset="TJA1050" device="" value="TJA1050"/>
 <part name="U$12" library="SchlegelAr_Master" deviceset="+5V" device=""/>
 <part name="GND21" library="supply1" deviceset="GND" device=""/>
@@
 <part name="C17" library="SchlegelAr_Master" deviceset="C_POL" device="4X4MM" value="10u"/>
 <part name="U$1" library="SchlegelAr_Master" deviceset="GND" device=""/>
+<part name="FRAME3" library="frames" deviceset="A4L-LOC" device=""/>
+<part name="D1" library="SchlegelAr_Master" deviceset="BZG03C15TR3" device="" value="Z3V6"/>
 </parts>
 <sheets>
+<sheet>
+<plain>
+<rectangle x1="40.64" y1="55.88" x2="88.9" y2="147.32" layer="91"/>
+<rectangle x1="96.52" y1="60.96" x2="119.38" y2="78.74" layer="91"/>
+<rectangle x1="96.52" y1="86.36" x2="119.38" y2="104.14" layer="91"/>
+<text x="101.6" y="63.5" size="3.81" layer="94">CAN0</text>
+<text x="101.6" y="88.9" size="3.81" layer="94">CAN1</text>
+<text x="60.96" y="58.42" size="3.81" layer="94">CPU</text>
+<text x="99.06" y="124.46" size="3.81" layer="94">FTDI</text>
+<text x="76.2" y="134.62" size="1.6764" layer="92">FTDI_RX</text>
+<text x="76.2" y="132.08" size="1.6764" layer="92">FTDI_TX</text>
+<text x="99.06" y="134.62" size="1.6764" layer="92">TXD</text>
+<text x="99.06" y="132.08" size="1.6764" layer="92">RXD</text>
+<text x="78.74" y="99.06" size="1.6764" layer="92">CAN0RX</text>
+<text x="78.74" y="73.66" size="1.6764" layer="92">CAN1RX</text>
+<text x="78.74" y="96.52" size="1.6764" layer="92">CAN0TX</text>
+<text x="78.74" y="71.12" size="1.6764" layer="92">CAN1TX</text>
+<text x="99.06" y="99.06" size="1.6764" layer="92">RX</text>
+<text x="99.06" y="96.52" size="1.6764" layer="92">TX</text>
+<text x="99.06" y="71.12" size="1.6764" layer="92">TX</text>
+<text x="99.06" y="73.66" size="1.6764" layer="92">RX</text>
+<text x="111.76" y="99.06" size="1.6764" layer="92">CANH</text>
+<text x="111.76" y="73.66" size="1.6764" layer="92">CANH</text>
+<text x="111.76" y="96.52" size="1.6764" layer="92">CANL</text>
+<text x="111.76" y="71.12" size="1.6764" layer="92">CANL</text>
+<rectangle x1="96.52" y1="121.92" x2="119.38" y2="139.7" layer="91"/>
+</plain>
+<instances>
+<instance part="FRAME3" gate="G$1" x="0" y="0"/>
+</instances>
+<busses>
+<bus name="B$3">
+<segment>
+<wire x1="88.9" y1="99.06" x2="96.52" y2="99.06" width="0.762" layer="92"/>
+</segment>
+</bus>
+<bus name="B$4">
+<segment>
+<wire x1="88.9" y1="96.52" x2="96.52" y2="96.52" width="0.762" layer="92"/>
+</segment>
+</bus>
+<bus name="B$5">
+<segment>
+<wire x1="88.9" y1="73.66" x2="96.52" y2="73.66" width="0.762" layer="92"/>
+</segment>
+</bus>
+<bus name="B$6">
+<segment>
+<wire x1="88.9" y1="71.12" x2="96.52" y2="71.12" width="0.762" layer="92"/>
+</segment>
+</bus>
+<bus name="B$1">
+<segment>
+<wire x1="88.9" y1="134.62" x2="96.52" y2="134.62" width="0.762" layer="92"/>
+</segment>
+</bus>
+<bus name="B$2">
+<segment>
+<wire x1="88.9" y1="132.08" x2="96.52" y2="132.08" width="0.762" layer="92"/>
+</segment>
+</bus>
+</busses>
+<nets>
+</nets>
+</sheet>
 <sheet>
 <plain>
@@
 <instance part="GND10" gate="1" x="228.6" y="40.64"/>
 <instance part="GND11" gate="1" x="238.76" y="40.64"/>
-<instance part="P+1" gate="1" x="142.24" y="66.04"/>
+<instance part="P+1" gate="1" x="149.86" y="63.5"/>
 <instance part="GND9" gate="1" x="137.16" y="7.62"/>
 <instance part="GND12" gate="1" x="142.24" y="7.62"/>
-<instance part="GND13" gate="1" x="152.4" y="7.62"/>
+<instance part="GND13" gate="1" x="149.86" y="7.62"/>
 <instance part="Q1" gate="G$1" x="208.28" y="106.68" rot="R90"/>
 <instance part="GND14" gate="1" x="220.98" y="96.52"/>
@@
 <instance part="C14" gate="G$1" x="215.9" y="101.6" rot="R180"/>
 <instance part="C11" gate="G$1" x="142.24" y="15.24" rot="R90"/>
-<instance part="C12" gate="G$1" x="152.4" y="15.24" rot="R90"/>
+<instance part="C12" gate="G$1" x="149.86" y="15.24" rot="R90"/>
 <instance part="P+2" gate="1" x="198.12" y="86.36"/>
 <instance part="P+3" gate="1" x="208.28" y="86.36"/>
@@
 <instance part="P+12" gate="1" x="30.48" y="38.1"/>
 <instance part="GND20" gate="1" x="50.8" y="15.24"/>
+<instance part="D1" gate="G$1" x="144.78" y="43.18" rot="R90"/>
 </instances>
 <busses>
@@
 </segment>
 <segment>
-<wire x1="152.4" y1="12.7" x2="152.4" y2="10.16" width="0.1524" layer="91"/>
+<wire x1="149.86" y1="12.7" x2="149.86" y2="10.16" width="0.1524" layer="91"/>
 <pinref part="GND13" gate="1" pin="GND"/>
 <pinref part="C12" gate="G$1" pin="P$1"/>
@@
 <segment>
 <pinref part="IC1" gate="G$9" pin="VDDIN_5"/>
-<wire x1="134.62" y1="35.56" x2="142.24" y2="35.56" width="0.1524" layer="91"/>
+<wire x1="134.62" y1="35.56" x2="149.86" y2="35.56" width="0.1524" layer="91"/>
 <pinref part="P+1" gate="1" pin="+5V"/>
-<wire x1="142.24" y1="35.56" x2="142.24" y2="55.88" width="0.1524" layer="91"/>
+<wire x1="149.86" y1="35.56" x2="149.86" y2="55.88" width="0.1524" layer="91"/>
 <pinref part="IC1" gate="G$9" pin="VDDIO3"/>
-<wire x1="142.24" y1="55.88" x2="142.24" y2="63.5" width="0.1524" layer="91"/>
+<wire x1="149.86" y1="55.88" x2="149.86" y2="60.96" width="0.1524" layer="91"/>
 <wire x1="134.62" y1="53.34" x2="137.16" y2="53.34" width="0.1524" layer="91"/>
 <wire x1="137.16" y1="53.34" x2="137.16" y2="55.88" width="0.1524" layer="91"/>
@@
 <wire x1="134.62" y1="55.88" x2="137.16" y2="55.88" width="0.1524" layer="91"/>
 <junction x="137.16" y="55.88"/>
-<wire x1="137.16" y1="55.88" x2="142.24" y2="55.88" width="0.1524" layer="91"/>
-<junction x="142.24" y="55.88"/>
+<wire x1="137.16" y1="55.88" x2="144.78" y2="55.88" width="0.1524" layer="91"/>
+<junction x="149.86" y="55.88"/>
+<pinref part="D1" gate="G$1" pin="C"/>
+<wire x1="144.78" y1="55.88" x2="149.86" y2="55.88" width="0.1524" layer="91"/>
+<wire x1="144.78" y1="45.72" x2="144.78" y2="55.88" width="0.1524" layer="91"/>
+<junction x="144.78" y="55.88"/>
 </segment>
 <segment>
@@
 <segment>
 <pinref part="IC1" gate="G$9" pin="VDDANA"/>
-<wire x1="134.62" y1="30.48" x2="152.4" y2="30.48" width="0.1524" layer="91"/>
-<wire x1="152.4" y1="30.48" x2="152.4" y2="20.32" width="0.1524" layer="91"/>
+<wire x1="134.62" y1="30.48" x2="149.86" y2="30.48" width="0.1524" layer="91"/>
+<wire x1="149.86" y1="30.48" x2="149.86" y2="20.32" width="0.1524" layer="91"/>
 <pinref part="C12" gate="G$1" pin="P$2"/>
 </segment>
@@
 </segment>
 </net>
+<net name="N$8" class="0">
+<segment>
+<pinref part="IC1" gate="G$9" pin="VDDIN_33"/>
+<pinref part="D1" gate="G$1" pin="A"/>
+<wire x1="134.62" y1="38.1" x2="144.78" y2="38.1" width="0.1524" layer="91"/>
+<wire x1="144.78" y1="38.1" x2="144.78" y2="40.64" width="0.1524" layer="91"/>
+</segment>
+</net>

Commit message: added embedded sw frame, started to work on port driver
Parts:
- added C18: 100n, SchlegelAr_Master:C_SMD0603
Connections:
- net GND: now also C18.P$1
- net N$8: now also C18.P$2
Changed lines of the file:
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@@
 <part name="FRAME3" library="frames" deviceset="A4L-LOC" device=""/>
 <part name="D1" library="SchlegelAr_Master" deviceset="BZG03C15TR3" device="" value="Z3V6"/>
+<part name="C18" library="SchlegelAr_Master" deviceset="C_SMD" device="0603" value="100n"/>
+<part name="GND23" library="supply1" deviceset="GND" device=""/>
 </parts>
 <sheets>
@@
 <instance part="GND20" gate="1" x="50.8" y="15.24"/>
 <instance part="D1" gate="G$1" x="144.78" y="43.18" rot="R90"/>
+<instance part="C18" gate="G$1" x="154.94" y="33.02" rot="R90"/>
+<instance part="GND23" gate="1" x="154.94" y="7.62"/>
 </instances>
 <busses>
@@
 <wire x1="50.8" y1="20.32" x2="50.8" y2="17.78" width="0.1524" layer="91"/>
 </segment>
+<segment>
+<pinref part="C18" gate="G$1" pin="P$1"/>
+<wire x1="154.94" y1="30.48" x2="154.94" y2="10.16" width="0.1524" layer="91"/>
+<pinref part="GND23" gate="1" pin="GND"/>
+</segment>
 </net>
 <net name="+5V" class="0">
@@
 <wire x1="134.62" y1="38.1" x2="144.78" y2="38.1" width="0.1524" layer="91"/>
 <wire x1="144.78" y1="38.1" x2="144.78" y2="40.64" width="0.1524" layer="91"/>
-</segment>
-</net>
+<pinref part="C18" gate="G$1" pin="P$2"/>
+<wire x1="144.78" y1="38.1" x2="154.94" y2="38.1" width="0.1524" layer="91"/>
+<junction x="144.78" y="38.1"/>
+</segment>
+</net>

Commit message: updated lbr AT32 package (wrong footprint used), added Dio driver, modified Port driver
Parts:
- IC1: device AT32UC3C264C:AT32UC3C264C -> AT32UC3C264C:AT32UC3C264C0.5MM
Changed lines of the file:
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@@
 </classes>
 <parts>
-<part name="IC1" library="AT32UC3C264C" deviceset="AT32UC3C264C" device=""/>
+<part name="IC1" library="AT32UC3C264C" deviceset="AT32UC3C264C" device="0.5MM"/>
 <part name="GND1" library="supply1" deviceset="GND" device=""/>
 <part name="GND2" library="supply1" deviceset="GND" device=""/>

Commit message: update
Connections:
- removed net N$1: C12.P$2, IC1G$9.VDDANA
- net +5V: now also C12.P$2, IC1G$9.VDDANA
Other:
- note added: "*NOTE: VDDANA, GNDANA need to be connected in order to use JTAG/aWire"
- moved on the sheet: C11, C12, C18, D1
Changed lines of the file:
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@@
 <plain>
 <text x="223.52" y="106.68" size="1.778" layer="91">Quarz: Farnell 2467824</text>
+<text x="147.32" y="27.94" size="1.778" layer="91">*NOTE: VDDANA, GNDANA need to be connected in order to use JTAG/aWire</text>
 </plain>
 <instances>
@@
 <instance part="IC1" gate="G$7" x="167.64" y="147.32"/>
 <instance part="IC1" gate="G$8" x="15.24" y="50.8"/>
-<instance part="IC1" gate="G$9" x="121.92" y="45.72"/>
+<instance part="IC1" gate="G$9" x="111.76" y="45.72"/>
 <instance part="GND1" gate="1" x="208.28" y="68.58"/>
 <instance part="GND2" gate="1" x="218.44" y="68.58"/>
@@
 <instance part="GND10" gate="1" x="228.6" y="40.64"/>
 <instance part="GND11" gate="1" x="238.76" y="40.64"/>
-<instance part="P+1" gate="1" x="149.86" y="63.5"/>
-<instance part="GND9" gate="1" x="137.16" y="7.62"/>
-<instance part="GND12" gate="1" x="142.24" y="7.62"/>
-<instance part="GND13" gate="1" x="149.86" y="7.62"/>
+<instance part="P+1" gate="1" x="139.7" y="63.5"/>
+<instance part="GND9" gate="1" x="127" y="7.62"/>
+<instance part="GND12" gate="1" x="132.08" y="7.62"/>
+<instance part="GND13" gate="1" x="139.7" y="7.62"/>
 <instance part="Q1" gate="G$1" x="208.28" y="106.68" rot="R90"/>
 <instance part="GND14" gate="1" x="220.98" y="96.52"/>
@@
 <instance part="C13" gate="G$1" x="215.9" y="111.76" rot="R180"/>
 <instance part="C14" gate="G$1" x="215.9" y="101.6" rot="R180"/>
-<instance part="C11" gate="G$1" x="142.24" y="15.24" rot="R90"/>
-<instance part="C12" gate="G$1" x="149.86" y="15.24" rot="R90"/>
+<instance part="C11" gate="G$1" x="132.08" y="15.24" rot="R90"/>
+<instance part="C12" gate="G$1" x="139.7" y="15.24" rot="R90"/>
 <instance part="P+2" gate="1" x="198.12" y="86.36"/>
 <instance part="P+3" gate="1" x="208.28" y="86.36"/>
@@
 <instance part="P+12" gate="1" x="30.48" y="38.1"/>
 <instance part="GND20" gate="1" x="50.8" y="15.24"/>
-<instance part="D1" gate="G$1" x="144.78" y="43.18" rot="R90"/>
-<instance part="C18" gate="G$1" x="154.94" y="33.02" rot="R90"/>
-<instance part="GND23" gate="1" x="154.94" y="7.62"/>
+<instance part="D1" gate="G$1" x="134.62" y="43.18" rot="R90"/>
+<instance part="C18" gate="G$1" x="144.78" y="33.02" rot="R90"/>
+<instance part="GND23" gate="1" x="144.78" y="7.62"/>
 </instances>
 <busses>
@@
 <segment>
 <pinref part="IC1" gate="G$9" pin="GNDIO1"/>
-<wire x1="134.62" y1="48.26" x2="137.16" y2="48.26" width="0.1524" layer="91"/>
-<wire x1="137.16" y1="48.26" x2="137.16" y2="45.72" width="0.1524" layer="91"/>
+<wire x1="124.46" y1="48.26" x2="127" y2="48.26" width="0.1524" layer="91"/>
+<wire x1="127" y1="48.26" x2="127" y2="45.72" width="0.1524" layer="91"/>
 <pinref part="IC1" gate="G$9" pin="GNDIO3"/>
-<wire x1="137.16" y1="45.72" x2="137.16" y2="43.18" width="0.1524" layer="91"/>
-<wire x1="137.16" y1="43.18" x2="134.62" y2="43.18" width="0.1524" layer="91"/>
+<wire x1="127" y1="45.72" x2="127" y2="43.18" width="0.1524" layer="91"/>
+<wire x1="127" y1="43.18" x2="124.46" y2="43.18" width="0.1524" layer="91"/>
 <pinref part="IC1" gate="G$9" pin="GNDIO2"/>
-<wire x1="134.62" y1="45.72" x2="137.16" y2="45.72" width="0.1524" layer="91"/>
-<junction x="137.16" y="45.72"/>
+<wire x1="124.46" y1="45.72" x2="127" y2="45.72" width="0.1524" layer="91"/>
+<junction x="127" y="45.72"/>
 <pinref part="IC1" gate="G$9" pin="GNDANA"/>
-<wire x1="134.62" y1="27.94" x2="137.16" y2="27.94" width="0.1524" layer="91"/>
-<wire x1="137.16" y1="27.94" x2="137.16" y2="20.32" width="0.1524" layer="91"/>
+<wire x1="124.46" y1="27.94" x2="127" y2="27.94" width="0.1524" layer="91"/>
+<wire x1="127" y1="27.94" x2="127" y2="20.32" width="0.1524" layer="91"/>
 <pinref part="IC1" gate="G$9" pin="GNDPLL"/>
-<wire x1="137.16" y1="20.32" x2="137.16" y2="15.24" width="0.1524" layer="91"/>
-<wire x1="137.16" y1="15.24" x2="137.16" y2="10.16" width="0.1524" layer="91"/>
-<wire x1="134.62" y1="15.24" x2="137.16" y2="15.24" width="0.1524" layer="91"/>
-<junction x="137.16" y="15.24"/>
+<wire x1="127" y1="20.32" x2="127" y2="15.24" width="0.1524" layer="91"/>
+<wire x1="127" y1="15.24" x2="127" y2="10.16" width="0.1524" layer="91"/>
+<wire x1="124.46" y1="15.24" x2="127" y2="15.24" width="0.1524" layer="91"/>
+<junction x="127" y="15.24"/>
 <pinref part="IC1" gate="G$9" pin="GNDCORE"/>
-<wire x1="134.62" y1="20.32" x2="137.16" y2="20.32" width="0.1524" layer="91"/>
-<junction x="137.16" y="20.32"/>
-<wire x1="137.16" y1="43.18" x2="137.16" y2="27.94" width="0.1524" layer="91"/>
-<junction x="137.16" y="43.18"/>
-<junction x="137.16" y="27.94"/>
+<wire x1="124.46" y1="20.32" x2="127" y2="20.32" width="0.1524" layer="91"/>
+<junction x="127" y="20.32"/>
+<wire x1="127" y1="43.18" x2="127" y2="27.94" width="0.1524" layer="91"/>
+<junction x="127" y="43.18"/>
+<junction x="127" y="27.94"/>
 <pinref part="GND9" gate="1" pin="GND"/>
 </segment>
 <segment>
-<wire x1="142.24" y1="12.7" x2="142.24" y2="10.16" width="0.1524" layer="91"/>
+<wire x1="132.08" y1="12.7" x2="132.08" y2="10.16" width="0.1524" layer="91"/>
 <pinref part="GND12" gate="1" pin="GND"/>
 <pinref part="C11" gate="G$1" pin="P$1"/>
 </segment>
 <segment>
-<wire x1="149.86" y1="12.7" x2="149.86" y2="10.16" width="0.1524" layer="91"/>
+<wire x1="139.7" y1="12.7" x2="139.7" y2="10.16" width="0.1524" layer="91"/>
 <pinref part="GND13" gate="1" pin="GND"/>
 <pinref part="C12" gate="G$1" pin="P$1"/>
@@
 <segment>
 <pinref part="C18" gate="G$1" pin="P$1"/>
-<wire x1="154.94" y1="30.48" x2="154.94" y2="10.16" width="0.1524" layer="91"/>
+<wire x1="144.78" y1="30.48" x2="144.78" y2="10.16" width="0.1524" layer="91"/>
 <pinref part="GND23" gate="1" pin="GND"/>
 </segment>
@@
 <segment>
 <pinref part="IC1" gate="G$9" pin="VDDIN_5"/>
-<wire x1="134.62" y1="35.56" x2="149.86" y2="35.56" width="0.1524" layer="91"/>
+<wire x1="124.46" y1="35.56" x2="139.7" y2="35.56" width="0.1524" layer="91"/>
 <pinref part="P+1" gate="1" pin="+5V"/>
-<wire x1="149.86" y1="35.56" x2="149.86" y2="55.88" width="0.1524" layer="91"/>
+<wire x1="139.7" y1="35.56" x2="139.7" y2="55.88" width="0.1524" layer="91"/>
 <pinref part="IC1" gate="G$9" pin="VDDIO3"/>
-<wire x1="149.86" y1="55.88" x2="149.86" y2="60.96" width="0.1524" layer="91"/>
-<wire x1="134.62" y1="53.34" x2="137.16" y2="53.34" width="0.1524" layer="91"/>
-<wire x1="137.16" y1="53.34" x2="137.16" y2="55.88" width="0.1524" layer="91"/>
+<wire x1="139.7" y1="55.88" x2="139.7" y2="60.96" width="0.1524" layer="91"/>
+<wire x1="124.46" y1="53.34" x2="127" y2="53.34" width="0.1524" layer="91"/>
+<wire x1="127" y1="53.34" x2="127" y2="55.88" width="0.1524" layer="91"/>
 <pinref part="IC1" gate="G$9" pin="VDDIO1"/>
-<wire x1="137.16" y1="55.88" x2="137.16" y2="58.42" width="0.1524" layer="91"/>
-<wire x1="134.62" y1="58.42" x2="137.16" y2="58.42" width="0.1524" layer="91"/>
+<wire x1="127" y1="55.88" x2="127" y2="58.42" width="0.1524" layer="91"/>
+<wire x1="124.46" y1="58.42" x2="127" y2="58.42" width="0.1524" layer="91"/>
 <pinref part="IC1" gate="G$9" pin="VDDIO2"/>
-<wire x1="134.62" y1="55.88" x2="137.16" y2="55.88" width="0.1524" layer="91"/>
-<junction x="137.16" y="55.88"/>
-<wire x1="137.16" y1="55.88" x2="144.78" y2="55.88" width="0.1524" layer="91"/>
-<junction x="149.86" y="55.88"/>
+<wire x1="124.46" y1="55.88" x2="127" y2="55.88" width="0.1524" layer="91"/>
+<junction x="127" y="55.88"/>
+<wire x1="127" y1="55.88" x2="134.62" y2="55.88" width="0.1524" layer="91"/>
+<junction x="139.7" y="55.88"/>
 <pinref part="D1" gate="G$1" pin="C"/>
-<wire x1="144.78" y1="55.88" x2="149.86" y2="55.88" width="0.1524" layer="91"/>
-<wire x1="144.78" y1="45.72" x2="144.78" y2="55.88" width="0.1524" layer="91"/>
-<junction x="144.78" y="55.88"/>
+<wire x1="134.62" y1="55.88" x2="139.7" y2="55.88" width="0.1524" layer="91"/>
+<wire x1="134.62" y1="45.72" x2="134.62" y2="55.88" width="0.1524" layer="91"/>
+<junction x="134.62" y="55.88"/>
+<pinref part="IC1" gate="G$9" pin="VDDANA"/>
+<wire x1="124.46" y1="30.48" x2="139.7" y2="30.48" width="0.1524" layer="91"/>
+<wire x1="139.7" y1="30.48" x2="139.7" y2="35.56" width="0.1524" layer="91"/>
+<junction x="139.7" y="35.56"/>
+<pinref part="C12" gate="G$1" pin="P$2"/>
+<wire x1="139.7" y1="30.48" x2="139.7" y2="20.32" width="0.1524" layer="91"/>
+<junction x="139.7" y="30.48"/>
 </segment>
 <segment>
@@
 <segment>
 <pinref part="IC1" gate="G$9" pin="VDDCORE"/>
-<wire x1="134.62" y1="22.86" x2="142.24" y2="22.86" width="0.1524" layer="91"/>
-<wire x1="142.24" y1="22.86" x2="142.24" y2="20.32" width="0.1524" layer="91"/>
+<wire x1="124.46" y1="22.86" x2="132.08" y2="22.86" width="0.1524" layer="91"/>
+<wire x1="132.08" y1="22.86" x2="132.08" y2="20.32" width="0.1524" layer="91"/>
 <pinref part="C11" gate="G$1" pin="P$2"/>
-</segment>
-</net>
-<net name="N$1" class="0">
-<segment>
-<pinref part="IC1" gate="G$9" pin="VDDANA"/>
-<wire x1="134.62" y1="30.48" x2="149.86" y2="30.48" width="0.1524" layer="91"/>
-<wire x1="149.86" y1="30.48" x2="149.86" y2="20.32" width="0.1524" layer="91"/>
-<pinref part="C12" gate="G$1" pin="P$2"/>
 </segment>
 </net>
@@
 <pinref part="IC1" gate="G$9" pin="VDDIN_33"/>
 <pinref part="D1" gate="G$1" pin="A"/>
+<wire x1="124.46" y1="38.1" x2="134.62" y2="38.1" width="0.1524" layer="91"/>
+<wire x1="134.62" y1="38.1" x2="134.62" y2="40.64" width="0.1524" layer="91"/>
+<pinref part="C18" gate="G$1" pin="P$2"/>
 <wire x1="134.62" y1="38.1" x2="144.78" y2="38.1" width="0.1524" layer="91"/>
-<wire x1="144.78" y1="38.1" x2="144.78" y2="40.64" width="0.1524" layer="91"/>
-<pinref part="C18" gate="G$1" pin="P$2"/>
-<wire x1="144.78" y1="38.1" x2="154.94" y2="38.1" width="0.1524" layer="91"/>
-<junction x="144.78" y="38.1"/>
-</segment>
-</net>
+<junction x="134.62" y="38.1"/>
+</segment>
+</net>

Commit message: sw modified
Parts:
- added C21: 100n, SchlegelAr_Master:C_SMD0603
Connections:
- net +5V: now also C21.P$2
- net GND: now also C21.P$1
Other:
- moved on the sheet: C11, C12, D1
