File: hw/CANSniftAndShift.brd (EAGLE design)
At the start: 160 x 100 mm, 41 parts, among them CON1 FCI-10033526-N3212LF, CON4 FCI-10033526-N3212LF, IC3 TJA1050, IC4 TJA1050, IC7 FT232RL, Q1 16MHz

Commit message: sw modified
Parts:
- added C21: 100n, SchlegelAr_Master:C0603
- moved R3 407.7 mm to (55.9, 80.0), turned to 270 degrees
- moved R2 392.6 mm to (24.1, 80.0), turned to 270 degrees
- moved JP3 391.3 mm to (54.6, 76.2), turned to 270 degrees
- moved X2 388.8 mm to (58.4, 83.8)
- moved JP2 382.3 mm to (25.4, 76.2), turned to 90 degrees
- moved X1 357.7 mm to (26.7, 83.8)
- moved IC4 307.2 mm to (40.6, 73.7)
- moved IC3 297.0 mm to (34.3, 73.7)
- moved CON1 265.1 mm to (57.1, 57.1), turned to 90 degrees
Connections:
- net +5V: now also C21.2
- net GND: now also C21.1
